Commit message: feat: add team UAV visual description

File: ros2_ws/src/racing_description/urdf/racing_uav.urdf.xacro (robot description, xacro)
@@ -4,5 +4,18 @@
   <xacro:arg name="camera_xyz" default="0.12 0.02 0.252"/>
   <xacro:arg name="camera_rpy" default="0 0 0"/>
-  <link name="base_link"/>
+  <!-- The detailed CAD mesh is visualization-only. Flight dynamics remain PX4-owned. -->
+  <link name="base_link">
+    <visual name="team_airframe_visual">
+      <origin xyz="0 0 0" rpy="0 0 0"/>
+      <geometry>
+        <mesh
+          filename="package://racing_description/meshes/team_racer/base_link.stl"
+          scale="1 1 1"/>
+      </geometry>
+      <material name="team_racer_gold">
+        <color rgba="0.64706 0.51765 0 1"/>
+      </material>
+    </visual>
+  </link>
   <link name="camera_link"/>
   <link name="camera_optical_frame"/>

Commit message: fix: align team UAV mesh with ROS axes

File: ros2_ws/src/racing_description/urdf/racing_uav.urdf.xacro (robot description, xacro)
@@ -7,5 +7,6 @@
   <link name="base_link">
     <visual name="team_airframe_visual">
-      <origin xyz="0 0 0" rpy="0 0 0"/>
+      <!-- Map SolidWorks Y-up axes to ROS X-forward, Y-left, Z-up axes. -->
+      <origin xyz="0 0 0" rpy="1.57079632679 0 1.57079632679"/>
       <geometry>
         <mesh
